Commit message: Interactive Gripper Control +

File: src/robotiq/cfg/s-model_articulated.urdf (robot description, URDF)
Before this commit: robot s-model_articulated, 13 links, 12 joints
Links:
- added link base_link
- link finger_1_link_0: mass None -> 1
- link finger_1_link_1: mass None -> 1
- link finger_1_link_2: mass None -> 1
- link finger_1_link_3: mass None -> 1
- link finger_2_link_0: mass None -> 1
- link finger_2_link_1: mass None -> 1
- link finger_2_link_2: mass None -> 1
- link finger_2_link_3: mass None -> 1
- link finger_middle_link_0: mass None -> 1
- link finger_middle_link_1: mass None -> 1
- link finger_middle_link_2: mass None -> 1
- link finger_middle_link_3: mass None -> 1
Joints:
- added joint base_link_palm_joint: type fixed, parent base_link, child palm

File: src/robotiq/cfg/s-model_articulated.xacro (robot description, xacro)
@@ -5,6 +5,6 @@
 -->
 <robot name="s-model_articulated" xmlns:xacro="http://ros.org/wiki/xacro">
-  <include filename="$(find robotiq)/cfg/s-model_articulated_macro.xacro" />
-  <xacro:s-model_articulated prefix=""/>
+    <include filename="$(find robotiq)/cfg/s-model_articulated_macro.xacro" />
+    <xacro:s-model_articulated prefix=""/>
 <!--
 	<include filename="$(find robotiq)/cfg/s-model_finger_articulated_macro.xacro" />
